File: Prj 3 - MCU Data Logger.kicad_pcb (KiCad board)
At the start: 4 copper layers, 49.6 x 35.6 mm, 29 parts, among them J1 Conn_01x04_Pin, J2 Conn_01x09_Pin, J3 Conn_01x04_Pin, J4 Conn_02x03_Odd_Even, U1 24LC1025, U2 24LC1025, U3 DS1337S_, U4 ATMEGA328P-AU, Y1 32.768 KHz, Y2 16MHz

Commit message: Fixed all bugs in 4layer PCB
Connections:
- J1 pad 4: /SCK -> /SCL
- R3 pad 2: /SCK -> /SCL
- U1 pad 6: /SCK -> /SCL
- U2 pad 6: /SCK -> /SCL
- U3 pad 6: /SCK -> /SCL
- U4 pad 28: /SCK -> /SCL
Routing:
- net /SCK: track 88.0 -> 24.9 mm, vias 7 -> 3
- net /SCL: track 0.00 -> 61.2 mm, vias 0 -> 5
- net /RESET: track 21.6 -> 23.8 mm
Other:
- board text added: "SCL"
- board text removed: "SCK"
